File: MegaGRRLDesktop.brd (EAGLE design)
At the start: 124.5 x 124.5 mm, 134 parts, among them IC1 UA78M33CKCS, IC10 PCA9634D, IC11 TPA6111A2DR, IC12 ESP-WROOM-32ESP-WROOM-32-NO-RF, IC14 CH340G, IC2 74HC595N, IC3 74HC595N, IC4 MCP23017SP, IC5 NE5532N, IC6 7805TV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

Commit message: fix 74HCT595
Parts:
- IC2, IC3: value 74HC595N -> 74HCT595N
Changed lines of the file:
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@@
 <attribute name="SPICEPREFIX" value="C" x="196.85" y="44.45" size="1.778" layer="27" rot="R90" display="off"/>
 </element>
-<element name="IC2" library="74xx-eu" library_urn="urn:adsk.eagle:library:85" package="DIL16" package3d_urn="urn:adsk.eagle:package:922/2" value="74HC595N" x="113.03" y="64.135" smashed="yes">
+<element name="IC2" library="74xx-eu" library_urn="urn:adsk.eagle:library:85" package="DIL16" package3d_urn="urn:adsk.eagle:package:922/2" value="74HCT595N" x="113.03" y="64.135" smashed="yes">
 <attribute name="NAME" x="102.87" y="60.96" size="1.27" layer="25" font="vector" ratio="10" rot="R90"/>
 <attribute name="POPULARITY" value="0" x="113.03" y="64.135" size="1.778" layer="27" display="off"/>
 </element>
-<element name="IC3" library="74xx-eu" library_urn="urn:adsk.eagle:library:85" package="DIL16" package3d_urn="urn:adsk.eagle:package:922/2" value="74HC595N" x="113.03" y="75.565" smashed="yes">
+<element name="IC3" library="74xx-eu" library_urn="urn:adsk.eagle:library:85" package="DIL16" package3d_urn="urn:adsk.eagle:package:922/2" value="74HCT595N" x="113.03" y="75.565" smashed="yes">
 <attribute name="NAME" x="102.87" y="70.485" size="1.27" layer="25" font="vector" ratio="10" rot="R90"/>
 <attribute name="POPULARITY" value="0" x="113.03" y="75.565" size="1.778" layer="27" display="off"/>
